File: mullet-pcb.kicad_pcb (KiCad board)
At the start: 2 copper layers, 299.7 x 97.7 mm, 187 parts, among them SW1 KEYSW, SW10 KEYSW, SW11 KEYSW, SW12 KEYSW, SW13 KEYSW, SW14 KEYSW, SW15 KEYSW, SW16 KEYSW, SW17 KEYSW, SW18 KEYSW, SW19 KEYSW, SW2 KEYSW, SW20 KEYSW, SW21 KEYSW, SW22 KEYSW, SW23 KEYSW, SW24 KEYSW, SW25 KEYSW, SW26 KEYSW, SW27 KEYSW, SW28 KEYSW, SW29 KEYSW, SW3 KEYSW, SW30 KEYSW, SW31 KEYSW, SW32 KEYSW, SW33 KEYSW, SW34 KEYSW, SW35 KEYSW, SW36 KEYSW, SW37 KEYSW, SW38 KEYSW, SW39 KEYSW, SW4 KEYSW, SW40 KEYSW, SW41 KEYSW, SW42 KEYSW, SW43 KEYSW, SW44 KEYSW, SW45 KEYSW, SW46 KEYSW, SW47 KEYSW, SW48 KEYSW, SW49 KEYSW, SW5 KEYSW, SW50 KEYSW, SW51 KEYSW, SW52 KEYSW, SW53 KEYSW, SW54 KEYSW, SW55 KEYSW, SW56 KEYSW, SW57 KEYSW, SW58 KEYSW, SW59 KEYSW, SW6 KEYSW, SW60 KEYSW, SW61 KEYSW, SW62 KEYSW, SW63 KEYSW, SW64 KEYSW, SW65 KEYSW, SW66 KEYSW, SW67 KEYSW, SW7 KEYSW, SW8 KEYSW, SW9 KEYSW, U1 ATMEGA32U4, U2 PRTR5V0U2X, X1 XTAL_GND

Commit message: clean up and remove unnecessary ground traces
Routing:
- net GND: track 1166.7 -> 1158.3 mm, vias 25 -> 24
- net row1: track 366.7 -> 362.8 mm

Commit message: curve traces
Parts:
- ISCP1: footprint keyboard_parts2:AVR_ICSP_3x2 -> keyboard_parts:AVR_ICSP_3x2
- R6: value 22Ω -> 22R
Routing:
- net GND: track 1158.3 -> 1096.9 mm, vias 24 -> 22
- net +5V: track 1040.1 -> 1019.4 mm
- net row0: track 370.5 -> 365.9 mm
- net row1: track 362.8 -> 358.3 mm
- net row4: track 349.0 -> 346.2 mm
- net row3: track 323.0 -> 320.4 mm
- net col4: track 179.3 -> 176.7 mm
- net col6: track 200.6 -> 198.6 mm
- net col13: track 340.5 -> 338.6 mm
- net Net-(C2-Pad1): track 10.1 -> 12.0 mm
- net col9: track 238.2 -> 236.4 mm
- net col3: track 142.5 -> 140.8 mm
- net col12: track 328.0 -> 326.3 mm
- net Net-(LED1-Pad2): track 50.5 -> 48.9 mm
- net col0: track 111.3 -> 109.9 mm
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- added copper zone on F.Cu, net GND
- removed copper zone on F.Cu, net (none)
Other:
- board text added: "500"
- board text added: "ESD"
- board text added: "mA"

Commit message: change page size
Parts:
- moved C1 111.7 mm to (86.7, 132.3)
- moved C11 111.7 mm to (291.2, 104.4)
- moved C13 111.7 mm to (176.9, 103.7)
- moved C15 111.7 mm to (77.1, 107.7)
- moved C19 111.7 mm to (206.2, 178.0)
- moved C20 111.7 mm to (253.2, 177.6)
- moved C3 111.7 mm to (93.6, 122.2)
- moved C6 111.7 mm to (99.1, 131.5)
- moved C9 111.7 mm to (359.4, 130.9)
- moved D11 111.7 mm to (260.6, 109.7)
- moved D15 111.7 mm to (355.8, 109.7)
- moved D17 111.7 mm to (109.9, 123.3)
- moved D18 111.7 mm to (112.6, 123.3)
- moved D30 111.7 mm to (350.3, 123.8)
- moved D46 111.7 mm to (113.0, 166.9)
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