File: mullet-pcb.kicad_pcb (KiCad board)
At the start: 2 copper layers, 299.7 x 97.7 mm, 187 parts, among them SW1 KEYSW, SW10 KEYSW, SW11 KEYSW, SW12 KEYSW, SW13 KEYSW, SW14 KEYSW, SW15 KEYSW, SW16 KEYSW, SW17 KEYSW, SW18 KEYSW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

Commit message: Update mullet-pcb.kicad_pcb
Routing:
- net GND: track 1096.9 -> 1099.8 mm, vias 22 -> 24
- net +5V: track 1019.1 -> 1018.6 mm
