File: mullet-pcb.kicad_pcb (KiCad board)
At the start: 2 copper layers, 299.7 x 97.7 mm, 187 parts, among them SW1 KEYSW, SW10 KEYSW, SW11 KEYSW, SW12 KEYSW, SW13 KEYSW, SW14 KEYSW, SW15 KEYSW, SW16 KEYSW, SW17 KEYSW, SW18 KEYSW, SW19 KEYSW, SW2 KEYSW, SW20 KEYSW, SW21 KEYSW, SW22 KEYSW, SW23 KEYSW, SW24 KEYSW, SW25 KEYSW, SW26 KEYSW, SW27 KEYSW, SW28 KEYSW, SW29 KEYSW, SW3 KEYSW, SW30 KEYSW, SW31 KEYSW, SW32 KEYSW, SW33 KEYSW, SW34 KEYSW, SW35 KEYSW, SW36 KEYSW, SW37 KEYSW, SW38 KEYSW, SW39 KEYSW, SW4 KEYSW, SW40 KEYSW, SW41 KEYSW, SW42 KEYSW, SW43 KEYSW, SW44 KEYSW, SW45 KEYSW, SW46 KEYSW, SW47 KEYSW, SW48 KEYSW, SW49 KEYSW, SW5 KEYSW, SW50 KEYSW, SW51 KEYSW, SW52 KEYSW, SW53 KEYSW, SW54 KEYSW, SW55 KEYSW, SW56 KEYSW, SW57 KEYSW, SW58 KEYSW, SW59 KEYSW, SW6 KEYSW, SW60 KEYSW, SW61 KEYSW, SW62 KEYSW, SW63 KEYSW, SW64 KEYSW, SW65 KEYSW, SW66 KEYSW, SW67 KEYSW, SW7 KEYSW, SW8 KEYSW, SW9 KEYSW, U1 ATMEGA32U4, U2 PRTR5V0U2X, X1 XTAL_GND

Commit message: update case, add footprint library, add teardrops
Parts:
- removed the G*** at (178.5, 177.3) (x2)
- removed MULLETFRONT: LOGO, logos:MULLET 9MM FMASK
- removed ST62: KEYSW, keyboard_parts2:Mx_Stab_625
- added G***: LOGO, logos:BOBBYHILL-HEAD 11MM, B.Cu at (221.0, 181.2)
- added G*** (x2): LOGO, logos:CFTKB_10MM_MASK, B.Cu at (210.5, 181.2)
- added G*** (x2): LOGO, logos:CFTKB_10MM_MASK, F.Cu at (165.6, 180.6)
- added G***: LOGO, logos:BOBBYHILL-HEAD 11MM, F.Cu at (155.1, 180.6)
- R6: value 22R -> 22
- SW62: footprint Button_Switch_Keyboard:SW_Cherry_MX1A_1.00u_PCB-NOSCREEN -> Button_Switch_Keyboard:SW_Cherry_MX_6.25u_PCB_ReversedStabilizer
- moved C11 6.38 mm to (285.8, 107.8)
- moved C19 6.38 mm to (200.9, 181.4)
- moved C22 6.38 mm to (342.8, 182.5)
- moved C9 6.38 mm to (354.0, 134.3)
- moved D11 6.38 mm to (255.2, 113.1)
- moved D15 6.38 mm to (350.4, 113.1)
- moved D34 6.38 mm to (136.0, 151.2)
- moved D36 6.38 mm to (174.1, 151.2)
- moved D41 6.38 mm to (269.4, 151.2)
- moved D42 6.38 mm to (288.4, 151.2)
- moved D43 6.38 mm to (319.4, 151.2)
- moved D44 6.38 mm to (350.4, 151.2)
- moved D49 6.38 mm to (164.7, 170.3)
- moved D52 6.38 mm to (222.2, 170.3)
- moved D55 6.38 mm to (279.0, 170.3)
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Connections:
- LED10 pad 2: Net-(LED10-Pad2) -> +5V
- LED10 pad 4: Net-(LED10-Pad4) -> +5V
- LED11 pad 2: Net-(LED11-Pad2) -> +5V
- LED11 pad 4: Net-(LED10-Pad2) -> +5V
- LED12 pad 2: Net-(LED12-Pad2) -> +5V
- LED12 pad 4: Net-(LED11-Pad2) -> +5V
- LED13 pad 2: Net-(LED13-Pad2) -> +5V
- LED13 pad 4: Net-(LED12-Pad2) -> +5V
- LED14 pad 4: Net-(LED13-Pad2) -> +5V
- LED9 pad 2: Net-(LED10-Pad4) -> +5V
Routing:
- net +5V: track 1018.4 -> 1275.5 mm
- net Net-(LED10-Pad2): track 66.5 -> 0.00 mm
- net Net-(LED10-Pad4): track 52.7 -> 0.00 mm
- net Net-(LED11-Pad2): track 46.1 -> 0.00 mm
- net Net-(LED12-Pad2): track 46.0 -> 0.00 mm
- net Net-(LED13-Pad2): track 45.9 -> 0.00 mm
- net col0: track 109.7 -> 108.0 mm
- net row1: track 358.2 -> 357.1 mm
- net GND: track 1099.7 -> 1100.4 mm
- added copper zone on B.Cu, net col0
- added copper zone on F.Cu, net col6
Other:
- board text added: "ISP"
- board text added: "M U L L E T"
- board text added: "coseyfannitutti 2019"
- board text removed: "MULLET"
- board text removed: "coseyfannitutti"
